File: roland_121_vcf_with_12db.brd (EAGLE design)
At the start: 100 x 80 mm, 89 parts, among them IC1 TL072P, IC2 LM13700N, IC3 LM13700N, Q1 MPF102, Q2 2N3904, Q3 2N3906, Q4 MPF102, Q6 MPF102, Q7 MPF102, Q8 2N3904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

Commit message: layout progress
Parts:
- removed C19: 22uF, rcl:B45181A
- added C11: 22uF, rcl:B45181A
- moved C18 171.6 mm to (-94.0, 58.4), turned to 0 degrees
- moved C6 164.1 mm to (-88.9, 47.0)
- moved R37 163.0 mm to (-58.4, 92.7), turned to 0 degrees
- moved R58 156.8 mm to (-58.4, 102.9)
- moved C17 156.4 mm to (-83.8, 58.4)
- moved C7 147.7 mm to (-95.2, 47.0), turned to 0 degrees
- moved 24DB_OUT 145.4 mm to (-85.1, 102.9)
- moved R34 145.1 mm to (-27.9, 92.7), turned to 0 degrees
- moved C5 138.8 mm to (-82.5, 47.0), turned to 0 degrees
- moved R30 136.9 mm to (-68.6, 87.6)
- moved R15 107.6 mm to (-88.9, 77.5), turned to 0 degrees
- moved C8 99.7 mm to (-16.5, 59.7), turned to 0 degrees
- moved R19 89.3 mm to (-38.1, 82.5), turned to 0 degrees
- moved D2 86.4 mm to (-53.3, 67.3), turned to 0 degrees
- moved C20 83.8 mm to (-21.6, 66.0), turned to 0 degrees
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Connections:
- removed net N$36: C19.-, C20.-
- new net N$30: C11.-, C20.-
- net N$14: now also IC2.16; no longer IC3.1
- net N$15: now also IC2.13; no longer IC3.4
- net N$2: now also IC3.1; no longer IC2.16
- net N$24: now also IC2.14; no longer IC3.3
- net N$3: now also IC3.4; no longer IC2.13
- net N$4: now also IC3.3; no longer IC2.14
- net N$41: now also IC3.5; no longer IC2.12
- net N$42: now also IC2.12; no longer IC3.5
- net N$60: now also C11.+; no longer C19.+
Routing:
- net GND: track 0.00 -> 12.7 mm
- net -12V: track 0.00 -> 2.54 mm
- net +12V: track 0.00 -> 2.54 mm
