File: roland_121_vcf_with_12db.sch (EAGLE design)
At the start: 97 parts, among them IC1 LM13700N, IC2 LM13700N, IC3 TL072P, Q1 2N3904, Q2 2N3906, Q3 2N3904, Q4 2N3904, Q5 MPF102, Q6 MPF102, Q7 MPF102, Q8 MPF102

Commit message: working on layout
Parts:
- removed 12DB_OUT: LSP10, solpad:LSP10
- removed C11, C12, C13, C14: 22uF, rcl:CPOL-USB45181A
- removed Q5: MPF102, mes_transistors:MPF102
- removed R1, R7: 100k, rcl:R-US_0207/7
- removed R18: 10k, rcl:R-US_0207/7
- removed R2, R3: 15k, rcl:R-US_0207/7
- removed R4: 560, rcl:R-US_0207/7
- removed R41: 68k, rcl:R-US_0207/7
- removed R44: 470k, rcl:R-US_0207/7
- removed R45: 47k, rcl:R-US_0207/7
- removed R46: 12k, rcl:R-US_0207/7
- added C19, C20: 22uF, rcl:CPOL-USB45181A
- added FREQ_TRIM: 100k, rcl:R-TRIMM64W
- added R53: 560, rcl:R-US_0207/7
- added R55: 68k, rcl:R-US_0207/7
- added R56: 15k, rcl:R-US_0207/7
- added R57: 22k, rcl:R-US_0207/7
- added WIDTH: 10k, rcl:R-TRIMM64W
- C10, C9: value 22uF -> 470p; device rcl:CPOL-USB45181A -> rcl:C-US025-030X050
- C15, C16: value 0.1uF -> 470p
- C17, C18: value 0.1uF -> 22uF; device rcl:C-US025-030X050 -> rcl:CPOL-USB45181A
- C2: value 470p -> 22uF; device rcl:C-US025-030X050 -> rcl:CPOL-USB45181A
- C3, C4, C5: value 470p -> 0.1uF
- C6, C7, C8: value 22uF -> 0.1uF; device rcl:CPOL-USB45181A -> rcl:C-US025-030X050
- IC1: value LM13700N -> TL072P; device synthdiy updated imperial:LM13700N -> linear:TL072P
- IC3: value TL072P -> LM13700N; device linear:TL072P -> synthdiy updated imperial:LM13700N
- Q1, Q4: value 2N3904 -> MPF102; device transistor-npn:2N3904 -> mes_transistors:MPF102
- Q2: value 2N3906 -> 2N3904; device transistor-pnp:2N3906 -> transistor-npn:2N3904
- Q3: value 2N3904 -> 2N3906; device transistor-npn:2N3904 -> transistor-pnp:2N3906
- Q8: value MPF102 -> 2N3904; device mes_transistors:MPF102 -> transistor-npn:2N3904
- R10: value 33k -> 100k
- R11, R30: value 15k -> 100k
- R12: value 10k -> 1M
- R13: value 10k -> 290k; device rcl:R-TRIMM64W -> rcl:R-US_0207/7
- R15: value 290k -> 10k
- R16: value 100k -> 15k; device rcl:R-TRIMM64W -> rcl:R-US_0207/7
- R17: value 1M -> 27k
- R19: value 1k8 -> 33k
- R20: value 5k6 -> 560
- R22: value 1k5 -> 560
- R23: value 100k -> 1k8
- R24: value 560 -> 5k6
- R25, R37: value 560 -> 10k
- R27: value 22k -> 15k
- R28: value 68k -> 1k5
- R31: value 560 -> 68k
- R33, R40: value 68k -> 560
- R34: value 22k -> 6k8
- R35: value 15k -> 68k
- R36: value 560 -> 15k
- R38: value 68k -> 22k
- R39: value 22k -> 68k
- R42: value 68k -> 100
- R43: value 4k7 -> 560
- R48: value 100k -> 10k
- R49: value 100 -> 68k
- R5: value 560 -> 100k
- R50: value 10k -> 15k
- R51: value 10k -> 22k
- R52: value 6k8 -> 68k
- R54: value 150k -> 560
- R9: value 27k -> 150k
- renumbered R47 to R58, U$1 to U1
Connections:
- removed net N$30: 12DB_OUT.MP, C10.+
- removed net N$31: Q3.E, R43.1
- removed net N$32: C7.+, Q3.C, R46.2
- removed net N$33: C11.+, Q3.B, R44.2, R45.1
- removed net N$35: C14.+, C8.+, Q4.E, R38.1, R58.2
- removed net N$37: C10.-, C7.-
- removed net N$38: C11.-, C6.-
- new net N$60: C17.+, C19.+, Q8.E, R55.1, R58.2
- net +12V: now also C3.1, C5.1, C7.1, FREQ_TRIM.E, IC1P.V+, IC3G$5.V+, Q1.D, Q2.C, Q4.D, Q8.C; no longer C15.1, C17.1, IC1G$5.V+, Q1.C, Q4.C, Q5.D, Q8.D, R16.E, R44.1, R46.1
- net -12V: now also C4.2, C6.2, C8.2, FREQ_TRIM.A, IC1P.V-, IC3G$5.V-, R13.2, R30.2, R38.1, R51.1, R57.1; no longer C16.2, C18.2, IC1G$5.V-, R15.2, R16.A, R23.2, R27.1, R34.1, R39.1, R43.2, R45.2
- net GND: now also C10.2, C16.2, C4.1, C6.1, C7.2, C8.1, C9.2, IC3G$3.IN, IC3G$4.IN, Q3.E, R15.2, R20.1, R22.1, R28.2, R33.1, R37.2, R40.1, R42.2, R43.1, R53.1, R54.1; no longer C16.1, C17.2, C18.1, C2.2, C4.2, IC1G$3.IN, IC1G$4.IN, Q2.E, R18.2, R22.2, R24.1, R25.1, R31.1, R36.1, R37.1, R4.1, R49.2, R5.1, R50.2
- net N$1: now also IC2A.IABC, R27.2; no longer IC1A.IABC, R2.2
- net N$10: now also R11.2; no longer R8.2
- net N$11: now also IC1A.+IN; no longer IC3A.+IN
- net N$12: now also IC1B.+IN, R15.1; no longer IC3B.+IN, R18.1
- net N$13: now also IC1B.OUT, R21.2, WIDTH.A, WIDTH.S; no longer IC3B.OUT, R12.2, R13.A, R13.S
- net N$14: now also IC3A.IABC, R50.2; no longer IC2A.IABC, R30.2
- net N$15: now also IC3A.-IN, R39.1, R40.2, R49.2; no longer IC2A.-IN, R32.2, R33.2, R41.1
- net N$16: now also IC1B.-IN, R10.1, R11.1, R12.1, R13.1, R16.2, R9.1; no longer IC3B.-IN, R11.2, R15.1, R17.1, R48.1, R54.1, R8.1
- net N$17: now also FREQ_TRIM.S, R12.2; no longer R16.S, R17.2
- net N$18: now also R23.1, R25.2; no longer R19.1, R21.2
- net N$19: now also R21.1, R23.2, R24.2; no longer R12.1, R19.2, R20.2
- net N$2: now also IC2B.IABC, R36.2; no longer IC1B.IABC, R3.2
- net N$20: now also Q2.B, R24.1, R25.1, R28.1; no longer Q1.B, R20.1, R21.1, R22.1
- net N$21: now also Q2.E, Q3.B, R30.1; no longer Q1.E, Q2.B, R23.1
- net N$22: now also IC2A.-IN, R19.1, R20.2; no longer IC1A.-IN, R10.1, R25.2
- net N$23: now also IC2A.+IN, R22.2, R34.1; no longer IC1A.+IN, R24.2, R52.1
- net N$24: now also IC3A.+IN, R43.2; no longer IC2A.+IN, R31.2
- net N$25: now also IC3B.IABC, R56.2; no longer IC2B.IABC, R35.2
- net N$26: now also IC3B.-IN, R52.1, R53.2, R55.2; no longer IC2B.-IN, R37.2, R38.2, R42.1
- net N$27: now also IC3B.+IN, R54.2; no longer IC2B.+IN, R36.2
- net N$28: now also Q1.S, R29.2, R31.2; no longer Q6.S, R27.2, R40.2
- net N$29: now also C20.+; no longer C9.+
- net N$3: now also IC2B.-IN, R31.1, R32.2, R35.2; no longer IC1B.-IN, R28.2, R40.1, R5.2
- net N$36: now also C19.-, C20.-; no longer C8.-, C9.-
- net N$39: now also C2.-; no longer C12.-
- net N$4: now also IC2B.+IN, R33.2; no longer IC1B.+IN, R4.2
- net N$40: now also C9.1, IC2A.OUT, Q1.G; no longer C2.1, IC1A.OUT, Q6.G
- net N$41: now also C10.1, IC2B.OUT, Q4.G; no longer C3.1, IC1B.OUT, Q5.G
- net N$42: now also C15.1, IC3A.OUT, Q6.G; no longer C4.1, IC2A.OUT, Q7.G
- net N$43: now also C16.1, IC3B.OUT, Q7.G; no longer C5.1, IC2B.OUT, Q8.G
- net N$44: now also Q6.S, R49.1, R51.2, R52.2; no longer Q7.S, R33.1, R34.2, R42.2
- net N$45: now also Q3.C, R27.1, R36.1, R50.1, R56.1; no longer Q2.C, R2.1, R3.1, R30.1, R35.1
- net N$46: now also Q4.S, R35.1, R38.2, R39.2; no longer C6.+, Q5.S, R28.1, R29.2, R41.2
- net N$47: now also Q7.S, Q8.B, R57.2; no longer Q4.B, Q8.S, R39.2
- net N$48: now also R42.1; no longer R49.1
- net N$49: now also C17.-, C18.-; no longer C13.-, C14.-
- net N$5: now also IN2_LEVEL.S, R5.2; no longer IN1_LEVEL.S, R7.2
- net N$50: now also C18.+, R48.2; no longer C13.+, R51.2
- net N$51: now also R48.1; no longer R51.1
- net N$52: now also R34.2, R37.1; no longer R50.1, R52.2
- net N$53: now also R10.2; no longer R48.2
- net N$56: now also R9.2; no longer R54.2
- net N$57: now also IN1_LEVEL.S, R8.1; no longer IN2_LEVEL.S, R1.1
- net N$6: now also R5.1, R8.2; no longer R1.2, R7.1
- net N$7: now also C2.+, IC1A.-IN, R17.2; no longer C12.+, IC3A.-IN, R9.2
- net N$8: now also IC1A.OUT, R17.1, R19.2; no longer IC3A.OUT, R10.2, R9.1
- net N$9: now also R16.1, WIDTH.E; no longer R11.1, R13.E
Other:
- moved on the sheet: C15, C16, C3, C4, C5, IC2A, IC2B, IN1, IN1_LEVEL, IN2, IN2_LEVEL, Q6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

Commit message: layout progress
Parts:
- renumbered C19 to C11
Connections:
- net N$14: now also IC2B.IABC; no longer IC3A.IABC
- net N$15: now also IC2B.-IN; no longer IC3A.-IN
- net N$2: now also IC3A.IABC; no longer IC2B.IABC
- net N$24: now also IC2B.+IN; no longer IC3A.+IN
- net N$3: now also IC3A.-IN; no longer IC2B.-IN
- net N$4: now also IC3A.+IN; no longer IC2B.+IN
- net N$41: now also IC3A.OUT; no longer IC2B.OUT
- net N$42: now also IC2B.OUT; no longer IC3A.OUT
Other:
- moved on the sheet: IC2B, IC3A
Changed lines of the file:
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@@
 <?xml version="1.0" encoding="utf-8"?>
 <!DOCTYPE eagle SYSTEM "eagle.dtd">
-<eagle version="7.1.0">
+<eagle version="7.2.0">
 <drawing>
 <settings>
@@
 <part name="P-14" library="supply1" deviceset="-12V" device=""/>
 <part name="P+14" library="supply1" deviceset="+12V" device=""/>
-<part name="C19" library="rcl" deviceset="CPOL-US" device="B45181A" value="22uF"/>
 <part name="Q4" library="mes_transistors" deviceset="MPF102" device=""/>
 <part name="Q1" library="mes_transistors" deviceset="MPF102" device=""/>
@@
 <part name="C4" library="rcl" deviceset="C-US" device="025-030X050" value="0.1uF"/>
 <part name="GND8" library="supply1" deviceset="GND" device=""/>
+<part name="C11" library="rcl" deviceset="CPOL-US" device="B45181A" value="22uF"/>
 </parts>
 <sheets>
@@
 <instances>
 <instance part="IC2" gate="A" x="17.78" y="53.34"/>
-<instance part="IC2" gate="B" x="93.98" y="53.34"/>
+<instance part="IC3" gate="A" x="93.98" y="53.34"/>
 <instance part="IC2" gate="G$3" x="-43.18" y="119.38"/>
 <instance part="IC2" gate="G$4" x="-43.18" y="127"/>
-<instance part="IC3" gate="A" x="172.72" y="53.34"/>
+<instance part="IC2" gate="B" x="172.72" y="53.34"/>
 <instance part="IC3" gate="B" x="248.92" y="53.34"/>
 <instance part="IC3" gate="G$3" x="-43.18" y="111.76"/>
@@
 <instance part="P-14" gate="1" x="292.1" y="25.4"/>
 <instance part="P+14" gate="1" x="292.1" y="58.42"/>
-<instance part="C19" gate="G$1" x="307.34" y="40.64" rot="R90"/>
 <instance part="Q4" gate="1" x="124.46" y="53.34"/>
 <instance part="Q1" gate="1" x="48.26" y="53.34"/>
@@
 <instance part="C4" gate="G$1" x="15.24" y="109.22"/>
 <instance part="GND8" gate="1" x="2.54" y="111.76"/>
+<instance part="C11" gate="G$1" x="307.34" y="40.64" rot="R90"/>
 </instances>
 <busses>
@@
 <pinref part="R36" gate="G$1" pin="2"/>
 <wire x1="106.68" y1="45.72" x2="106.68" y2="43.18" width="0.1524" layer="91"/>
-<pinref part="IC2" gate="B" pin="IABC"/>
+<pinref part="IC3" gate="A" pin="IABC"/>
 </segment>
 </net>
@@
 <wire x1="76.2" y1="78.74" x2="76.2" y2="58.42" width="0.1524" layer="91"/>
 <junction x="76.2" y="58.42"/>
-<pinref part="IC2" gate="B" pin="-IN"/>
+<pinref part="IC3" gate="A" pin="-IN"/>
 <pinref part="R31" gate="G$1" pin="1"/>
 <junction x="71.12" y="58.42"/>
@@
 <wire x1="83.82" y1="48.26" x2="78.74" y2="48.26" width="0.1524" layer="91"/>
 <wire x1="78.74" y1="48.26" x2="78.74" y2="45.72" width="0.1524" layer="91"/>
-<pinref part="IC2" gate="B" pin="+IN"/>
+<pinref part="IC3" gate="A" pin="+IN"/>
 </segment>
 </net>
@@
 <pinref part="R50" gate="G$1" pin="2"/>
 <wire x1="185.42" y1="45.72" x2="185.42" y2="43.18" width="0.1524" layer="91"/>
-<pinref part="IC3" gate="A" pin="IABC"/>
+<pinref part="IC2" gate="B" pin="IABC"/>
 </segment>
 </net>
@@
 <wire x1="154.94" y1="78.74" x2="154.94" y2="58.42" width="0.1524" layer="91"/>
 <junction x="154.94" y="58.42"/>
-<pinref part="IC3" gate="A" pin="-IN"/>
+<pinref part="IC2" gate="B" pin="-IN"/>
 <pinref part="R39" gate="G$1" pin="1"/>
 <junction x="149.86" y="58.42"/>
@@
 <wire x1="162.56" y1="48.26" x2="157.48" y2="48.26" width="0.1524" layer="91"/>
 <wire x1="157.48" y1="48.26" x2="157.48" y2="45.72" width="0.1524" layer="91"/>
-<pinref part="IC3" gate="A" pin="+IN"/>
+<pinref part="IC2" gate="B" pin="+IN"/>
 </segment>
 </net>
@@
 </segment>
 </net>
-<net name="N$36" class="0">
-<segment>
-<pinref part="C19" gate="G$1" pin="-"/>
-<pinref part="C20" gate="G$1" pin="-"/>
-</segment>
-</net>
 <net name="N$39" class="0">
 <segment>
@@
 <net name="N$41" class="0">
 <segment>
-<pinref part="IC2" gate="B" pin="OUT"/>
+<pinref part="IC3" gate="A" pin="OUT"/>
 <pinref part="Q4" gate="1" pin="G"/>
 <wire x1="119.38" y1="53.34" x2="116.84" y2="53.34" width="0.1524" layer="91"/>
@@
 <net name="N$42" class="0">
 <segment>
-<pinref part="IC3" gate="A" pin="OUT"/>
+<pinref part="IC2" gate="B" pin="OUT"/>
 <pinref part="Q6" gate="1" pin="G"/>
 <wire x1="198.12" y1="53.34" x2="195.58" y2="53.34" width="0.1524" layer="91"/>
@@
 <net name="N$60" class="0">
 <segment>
-<pinref part="C19" gate="G$1" pin="+"/>
-<pinref part="C19" gate="G$1" pin="+"/>
 <pinref part="Q8" gate="G1" pin="E"/>
 <pinref part="R58" gate="G$1" pin="2"/>
@@
 <wire x1="299.72" y1="20.32" x2="299.72" y2="40.64" width="0.1524" layer="91"/>
 <junction x="299.72" y="40.64"/>
+<pinref part="C11" gate="G$1" pin="+"/>
 <wire x1="304.8" y1="40.64" x2="299.72" y2="40.64" width="0.1524" layer="91"/>
-<junction x="304.8" y="40.64"/>
-</segment>
-</net>
+</segment>
+</net>
+<net name="N$30" class="0">
+<segment>
+<pinref part="C20" gate="G$1" pin="-"/>
+<pinref part="C11" gate="G$1" pin="-"/>
+</segment>
+</net>
