File: eagle/roland_121_vcf.brd (EAGLE design)
At the start: 99.4 x 67.9 mm, 100 parts, among them IC1 TL072P, IC2 LM13700N, IC3 LM13700N, Q1 2SK30, Q2 2N3904, Q3 2N3906, Q4 2SK30, Q5 2N3904, Q6 2SK30, Q8 2N3904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

Commit message: fixed the wrong valued resistor
Parts:
- R52: value 68k -> 33k
Changed lines of the file:
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@@
 <attribute name="VALUE" x="83.2612" y="25.146" size="1.27" layer="27" ratio="10" rot="R270"/>
 </element>
-<element name="R52" library="rcl" package="0207/7" value="68k" x="82.55" y="45.72" smashed="yes" rot="R90">
+<element name="R52" library="rcl" package="0207/7" value="33k" x="82.55" y="45.72" smashed="yes" rot="R90">
 <attribute name="VALUE" x="83.1088" y="43.434" size="1.27" layer="27" ratio="10" rot="R90"/>
 </element>
